File: arduinomotorsturing/arduino_uno_r3_from_scratch-master/Driver.sch (KiCad schematic (older format))
At the start: 6 parts, among them U2 74HC1G04, U4 74HC1G04, U6 L298P

Commit message: sensor module
Parts:
- U2, U4: symbol 74HC1G04:74HC1G04 -> Arduino_Uno_R3_From_Scratch-rescue:74HC1G04-74HC1G04
Changed lines of the file:
@@
 $EndComp
 $Comp
-L 74HC1G04:74HC1G04 U4
+L Arduino_Uno_R3_From_Scratch-rescue:74HC1G04-74HC1G04 U4
 U 1 1 5BE4A21D
 P 7675 3775
@@
 $EndComp
 $Comp
-L 74HC1G04:74HC1G04 U2
+L Arduino_Uno_R3_From_Scratch-rescue:74HC1G04-74HC1G04 U2
 U 1 1 5BE4A42F
 P 2250 3775
