File: sensormodule_test_met2sensoren/sensormodule/sensormodule.kicad_pcb (KiCad board)
At the start: 2 copper layers, 9 parts, among them J1 Screw_Terminal_01x04, U1 QRE1113, U2 QRE1113

Commit message: sens
se
Other:
- board text added: "Vcc"
- board text added: "gnd"
Changed lines of the file:
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@@
   (general
     (thickness 1.6)
-    (drawings 0)
+    (drawings 2)
     (tracks 65)
     (zones 0)
@@
   )
   (setup
-    (last_trace_width 0.5)
+    (last_trace_width 0.25)
     (user_trace_width 0.5)
     (trace_clearance 0.2)
@@
     (pad_to_mask_clearance 0.2)
     (aux_axis_origin 0 0)
-    (visible_elements FFFFFF7F)
+    (visible_elements 7FFFFFFF)
     (pcbplotparams
       (layerselection 0x010fc_ffffffff)
@@
     )
   )
+  (gr_text Vcc (at 143.51 66.548) (layer F.Cu)
+    (effects (font (size 1 1) (thickness 0.25)))
+  )
+  (gr_text "gnd\n" (at 127 63.754) (layer F.Cu)
+    (effects (font (size 1.5 1.5) (thickness 0.3)))
+  )
   (segment (start 137.414 51.816) (end 134.747 54.483) (width 0.5) (layer F.Cu) (net 1))
