File: sensoren/sensormodule/sensormodule/sensormodule.kicad_pcb (KiCad board)
At the start: 2 copper layers, 12 parts, among them J1 Screw_Terminal_01x05, U1 QRE1113, U2 QRE1113, U3 QRE1113

Commit message: g
Parts:
- moved U1 11.7 mm to (120.0, 84.7)
- moved U3 8.34 mm to (160.0, 84.7)
- moved U2 1.66 mm to (140.0, 84.7)
Routing:
- net GND: track 61.2 -> 92.0 mm
- net Net-(R3-Pad2): track 31.7 -> 50.1 mm
- net Net-(J1-Pad2): track 16.8 -> 28.4 mm
- net Net-(R1-Pad2): track 8.14 -> 19.6 mm
- net Net-(J1-Pad4): track 22.1 -> 30.5 mm
- net Net-(R5-Pad2): track 15.5 -> 22.5 mm
- net Net-(J1-Pad3): track 27.5 -> 26.5 mm

Commit message: u
u
Routing:
- added copper zone on F.Cu, net GND
Changed lines of the file:
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@@
   )
   (setup
-    (last_trace_width 0.5)
+    (last_trace_width 0.25)
     (user_trace_width 0.5)
     (user_trace_width 1)
@@
   (segment (start 142 85.571) (end 140.871 85.571) (width 0.5) (layer F.Cu) (net 2))
   (segment (start 140.871 85.571) (end 139.071 83.771) (width 0.5) (layer F.Cu) (net 2))
-  (segment (start 138.346001 77.763001) (end 139.196 78.613) (width 0.5) (layer F.Cu) (net 3))
-  (segment (start 136.411347 75.828347) (end 138.346001 77.763001) (width 0.5) (layer F.Cu) (net 3))
-  (segment (start 133.068847 75.828347) (end 136.411347 75.828347) (width 0.5) (layer F.Cu) (net 3))
-  (segment (start 132.2975 75.057) (end 133.068847 75.828347) (width 0.5) (layer F.Cu) (net 3))
-  (segment (start 135.8535 67.564) (end 132.1705 71.247) (width 0.5) (layer F.Cu) (net 4))
-  (segment (start 140.208 67.564) (end 135.8535 67.564) (width 0.5) (layer F.Cu) (net 4))
-  (segment (start 140.843 68.199) (end 140.208 67.564) (width 0.5) (layer F.Cu) (net 4))
-  (segment (start 140.843 75.692) (end 140.843 68.199) (width 0.5) (layer F.Cu) (net 4))
-  (segment (start 141.736 78.613) (end 141.736 76.585) (width 0.5) (layer F.Cu) (net 4))
-  (segment (start 141.736 76.585) (end 140.843 75.692) (width 0.5) (layer F.Cu) (net 4))
-  (segment (start 141.736 83.507) (end 142 83.771) (width 0.5) (layer F.Cu) (net 4))
-  (segment (start 141.736 78.613) (end 141.736 83.507) (width 0.5) (layer F.Cu) (net 4))
-  (segment (start 144.4355 78.613) (end 144.276 78.613) (width 0.5) (layer F.Cu) (net 5))
-  (segment (start 150.6585 72.39) (end 144.4355 78.613) (width 0.5) (layer F.Cu) (net 5))
   (segment (start 146.786 83.771) (end 151.421 83.771) (width 0.5) (layer F.Cu) (net 2))
   (segment (start 142 85.571) (end 144.986 85.571) (width 0.5) (layer F.Cu) (net 2))
@@
   (segment (start 158 83.771) (end 158.571 83.771) (width 0.5) (layer F.Cu) (net 2))
   (segment (start 158.571 83.771) (end 160.371 85.571) (width 0.5) (layer F.Cu) (net 2))
+  (segment (start 138.346001 77.763001) (end 139.196 78.613) (width 0.5) (layer F.Cu) (net 3))
+  (segment (start 136.411347 75.828347) (end 138.346001 77.763001) (width 0.5) (layer F.Cu) (net 3))
+  (segment (start 133.068847 75.828347) (end 136.411347 75.828347) (width 0.5) (layer F.Cu) (net 3))
+  (segment (start 132.2975 75.057) (end 133.068847 75.828347) (width 0.5) (layer F.Cu) (net 3))
   (segment (start 127 83.771) (end 122 83.771) (width 0.5) (layer F.Cu) (net 3))
   (segment (start 135.304 83.771) (end 127 83.771) (width 0.5) (layer F.Cu) (net 3))
   (segment (start 139.196 78.613) (end 139.196 79.879) (width 0.5) (layer F.Cu) (net 3))
   (segment (start 139.196 79.879) (end 135.304 83.771) (width 0.5) (layer F.Cu) (net 3))
+  (segment (start 135.8535 67.564) (end 132.1705 71.247) (width 0.5) (layer F.Cu) (net 4))
+  (segment (start 140.208 67.564) (end 135.8535 67.564) (width 0.5) (layer F.Cu) (net 4))
+  (segment (start 140.843 68.199) (end 140.208 67.564) (width 0.5) (layer F.Cu) (net 4))
+  (segment (start 140.843 75.692) (end 140.843 68.199) (width 0.5) (layer F.Cu) (net 4))
+  (segment (start 141.736 78.613) (end 141.736 76.585) (width 0.5) (layer F.Cu) (net 4))
+  (segment (start 141.736 76.585) (end 140.843 75.692) (width 0.5) (layer F.Cu) (net 4))
+  (segment (start 141.736 83.507) (end 142 83.771) (width 0.5) (layer F.Cu) (net 4))
+  (segment (start 141.736 78.613) (end 141.736 83.507) (width 0.5) (layer F.Cu) (net 4))
+  (segment (start 144.4355 78.613) (end 144.276 78.613) (width 0.5) (layer F.Cu) (net 5))
+  (segment (start 150.6585 72.39) (end 144.4355 78.613) (width 0.5) (layer F.Cu) (net 5))
   (segment (start 160.67 83.771) (end 162 83.771) (width 0.5) (layer F.Cu) (net 5))
   (segment (start 159.068 82.169) (end 160.67 83.771) (width 0.5) (layer F.Cu) (net 5))
@@
   (segment (start 164.2 86.5) (end 163.4 87.3) (width 0.5) (layer F.Cu) (net 8))
   (segment (start 163.4 87.3) (end 159.8 87.3) (width 0.5) (layer F.Cu) (net 8))
+  (zone (net 2) (net_name GND) (layer F.Cu) (hatch edge 0.508)
+    (connect_pads (clearance 0.508))
+    (min_thickness 0.254)
+    (fill yes (arc_segments 16) (thermal_gap 0.508) (thermal_bridge_width 0.508))
+    (polygon
+      (pts
+        (xy 111.76 60.96) (xy 170.18 60.96) (xy 170.18 88.9) (xy 111.76 88.9)
+      )
+    )
+  )
 )

Commit message: todo code
Routing:
- added copper zone on F.Cu, net +5V
Other:
- board text added: "Billy was here"
Changed lines of the file:
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@@
   (general
     (thickness 1.6)
-    (drawings 17)
+    (drawings 18)
     (tracks 103)
     (zones 0)
@@
       (rotate (xyz 0 0 0))
     )
+  )
+  (gr_text "Billy was here\n" (at 139.625 63.2) (layer F.Cu)
+    (effects (font (size 1.5 1.5) (thickness 0.3)))
   )
   (gr_line (start 150.4 50) (end 150.4 55) (layer F.SilkS) (width 0.2))
@@
       )
     )
+  )
+  (zone (net 1) (net_name +5V) (layer F.Cu) (hatch edge 0.508)
+    (connect_pads (clearance 0.508))
+    (min_thickness 0.254)
+    (fill yes (arc_segments 16) (thermal_gap 0.508) (thermal_bridge_width 0.508))
+    (polygon
+      (pts
+        (xy 142.425 69.5) (xy 150.625 69.275) (xy 153.85 72.55) (xy 153.45 73.75) (xy 151.25 75.925)
+        (xy 150.7 77.35) (xy 150.725 79.7) (xy 150.1 79.475) (xy 149.875 78.9) (xy 148.975 78.625)
+        (xy 147.4 78.575) (xy 146.325 78.575) (xy 145.075 77.275) (xy 143.65 77) (xy 143.35 73.85)
+        (xy 143.425 72.475) (xy 143.35 70.6) (xy 142.675 69.525)
+      )
+    )
+  )
+  (zone (net 1) (net_name +5V) (layer F.Cu) (hatch edge 0.508)
+    (connect_pads (clearance 0.508))
+    (min_thickness 0.254)
+    (fill yes (arc_segments 16) (thermal_gap 0.508) (thermal_bridge_width 0.508))
+    (polygon
+      (pts
+        (xy 143.675 77.15) (xy 144.8 77.2) (xy 144.7 76.7) (xy 143.75 76.75) (xy 143.65 76.85)
+        (xy 143.65 77.075)
+      )
+    )
+  )
+  (zone (net 1) (net_name +5V) (layer F.Cu) (hatch edge 0.508)
+    (connect_pads (clearance 0.508))
+    (min_thickness 0.254)
+    (fill yes (arc_segments 16) (thermal_gap 0.508) (thermal_bridge_width 0.508))
+    (polygon
+      (pts
+        (xy 144.725 77.2) (xy 143.475 77.2) (xy 143.475 75.525) (xy 143.825 75.525)
+      )
+    )

Commit message: hey
Routing:
- net Net-(R3-Pad2): track 50.1 -> 53.1 mm
- net Net-(R5-Pad2): track 22.5 -> 23.8 mm
- removed copper zone on F.Cu, net GND
Changed lines of the file:
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@@
   (segment (start 161.408 88.392) (end 161 88.392) (width 0.5) (layer F.Cu) (net 7))
   (segment (start 161 88.392) (end 155.4 88.392) (width 0.5) (layer F.Cu) (net 7))
-  (segment (start 164.508 88.392) (end 161 88.392) (width 0.5) (layer F.Cu) (net 7))
-  (segment (start 165.7 87.2) (end 164.508 88.392) (width 0.5) (layer F.Cu) (net 7))
-  (segment (start 165.7 81.9) (end 165.7 87.2) (width 0.5) (layer F.Cu) (net 7))
-  (segment (start 161.8 78) (end 165.7 81.9) (width 0.5) (layer F.Cu) (net 7))
+  (segment (start 166.608 88.392) (end 161 88.392) (width 0.5) (layer F.Cu) (net 7))
+  (segment (start 167 88) (end 166.608 88.392) (width 0.5) (layer F.Cu) (net 7))
+  (segment (start 167 82) (end 167 88) (width 0.5) (layer F.Cu) (net 7))
+  (segment (start 163 78) (end 167 82) (width 0.5) (layer F.Cu) (net 7))
   (segment (start 153.6335 76.454) (end 155.1795 78) (width 0.5) (layer F.Cu) (net 7))
-  (segment (start 155.1795 78) (end 161.8 78) (width 0.5) (layer F.Cu) (net 7))
+  (segment (start 155.1795 78) (end 163 78) (width 0.5) (layer F.Cu) (net 7))
   (segment (start 158.071 85.571) (end 158 85.571) (width 0.5) (layer F.Cu) (net 8))
   (segment (start 159.8 87.3) (end 158.071 85.571) (width 0.5) (layer F.Cu) (net 8))
-  (segment (start 154.84151 80.96401) (end 161.96401 80.96401) (width 0.5) (layer F.Cu) (net 8))
+  (segment (start 154.84151 80.96401) (end 162.96401 80.96401) (width 0.5) (layer F.Cu) (net 8))
   (segment (start 153.6335 79.756) (end 154.84151 80.96401) (width 0.5) (layer F.Cu) (net 8))
-  (segment (start 161.96401 80.96401) (end 164.2 83.2) (width 0.5) (layer F.Cu) (net 8))
-  (segment (start 164.2 83.2) (end 164.2 86.5) (width 0.5) (layer F.Cu) (net 8))
-  (segment (start 164.2 86.5) (end 163.4 87.3) (width 0.5) (layer F.Cu) (net 8))
+  (segment (start 162.96401 80.96401) (end 165 83) (width 0.5) (layer F.Cu) (net 8))
+  (segment (start 165 83) (end 165 85.7) (width 0.5) (layer F.Cu) (net 8))
+  (segment (start 165 85.7) (end 163.4 87.3) (width 0.5) (layer F.Cu) (net 8))
   (segment (start 163.4 87.3) (end 159.8 87.3) (width 0.5) (layer F.Cu) (net 8))
-  (zone (net 2) (net_name GND) (layer F.Cu) (hatch edge 0.508)
-    (connect_pads (clearance 0.508))
-    (min_thickness 0.254)
-    (fill yes (arc_segments 16) (thermal_gap 0.508) (thermal_bridge_width 0.508))
-    (polygon
-      (pts
-        (xy 111.76 60.96) (xy 170.18 60.96) (xy 170.18 88.9) (xy 111.76 88.9)
-      )
-    )
-  )
   (zone (net 1) (net_name +5V) (layer F.Cu) (hatch edge 0.508)
     (connect_pads (clearance 0.508))
     (min_thickness 0.254)
-    (fill yes (arc_segments 16) (thermal_gap 0.508) (thermal_bridge_width 0.508))
+    (fill (arc_segments 16) (thermal_gap 0.508) (thermal_bridge_width 0.508))
     (polygon
       (pts
@@
     (connect_pads (clearance 0.508))
     (min_thickness 0.254)
-    (fill yes (arc_segments 16) (thermal_gap 0.508) (thermal_bridge_width 0.508))
+    (fill (arc_segments 16) (thermal_gap 0.508) (thermal_bridge_width 0.508))
     (polygon
       (pts
@@
     (connect_pads (clearance 0.508))
     (min_thickness 0.254)
-    (fill yes (arc_segments 16) (thermal_gap 0.508) (thermal_bridge_width 0.508))
+    (fill (arc_segments 16) (thermal_gap 0.508) (thermal_bridge_width 0.508))
     (polygon
       (pts
