File: pcbProject/IOExpander.sch (KiCad schematic (older format))
At the start: 3 parts

Commit message: bestellijst+pcbvoltageregulator aangepast
Parts:
- IO_EXPANDER_IC1, IO_EXPANDER_IC2: footprint SOP65P640X120-16N -> TCA9554PWR:SOP65P640X120-16N
Changed lines of the file:
@@
 F 0 "IO_EXPANDER_IC1" H 3675 4645 50  0000 C CNN
 F 1 "TCA9554PWR" H 3675 4554 50  0000 C CNN
-F 2 "SOP65P640X120-16N" H 3675 3875 50  0001 L BNN
+F 2 "TCA9554PWR:SOP65P640X120-16N" H 3675 3875 50  0001 L BNN
 F 3 "TCA9554PWR" H 3675 3875 50  0001 L BNN
 F 4 "296-30135-1-ND" H 3675 3875 50  0001 L BNN "Field4"
@@
 F 0 "IO_EXPANDER_IC2" H 6375 4670 50  0000 C CNN
 F 1 "TCA9554PWR" H 6375 4579 50  0000 C CNN
-F 2 "SOP65P640X120-16N" H 6375 3900 50  0001 L BNN
+F 2 "TCA9554PWR:SOP65P640X120-16N" H 6375 3900 50  0001 L BNN
 F 3 "TCA9554PWR" H 6375 3900 50  0001 L BNN
 F 4 "296-30135-1-ND" H 6375 3900 50  0001 L BNN "Field4"
@@
 F 0 "IO_Expander1" H 8203 4191 50  0000 L CNN
 F 1 "CONN_01X08" H 8203 4100 50  0000 L CNN
-F 2 "" H 8125 4150 60  0000 C CNN
+F 2 "" H 8125 4150 60  0001 C CNN
 F 3 "" H 8125 4150 60  0000 C CNN
 	1    8125 4150

Commit message: deel1routingpcb
Parts:
- IO_Expander1: footprint (none) -> Connector_PinSocket_2.54mm:PinSocket_1x08_P2.54mm_Vertical
Changed lines of the file:
@@
 F 0 "IO_Expander1" H 8203 4191 50  0000 L CNN
 F 1 "CONN_01X08" H 8203 4100 50  0000 L CNN
-F 2 "" H 8125 4150 60  0001 C CNN
+F 2 "Connector_PinSocket_2.54mm:PinSocket_1x08_P2.54mm_Vertical" H 8125 4150 60  0001 C CNN
 F 3 "" H 8125 4150 60  0000 C CNN
 	1    8125 4150
