File: pcbProject/MotorDriver.sch (KiCad schematic (older format))
At the start: 2 parts

Commit message: schema Afgewerkt
Changed lines of the file:
@@
 Text HLabel 4350 3150 2    50   Input ~ 0
 A01
-Wire Wire Line
-	4100 3150 4200 3150
-Wire Wire Line
-	4200 3150 4200 3250
-Wire Wire Line
-	4200 3250 4100 3250
-Connection ~ 4200 3150
-Wire Wire Line
-	4200 3150 4350 3150
 Text HLabel 4350 3350 2    50   Input ~ 0
 A02
 Wire Wire Line
-	4100 3350 4200 3350
-Wire Wire Line
 	4100 3450 4200 3450
-Wire Wire Line
-	4200 3450 4200 3350
-Connection ~ 4200 3350
-Wire Wire Line
-	4200 3350 4350 3350
 Text HLabel 4350 3650 2    50   Input ~ 0
 B01
-Wire Wire Line
-	4100 3650 4200 3650
-Wire Wire Line
-	4100 3750 4200 3750
-Wire Wire Line
-	4200 3750 4200 3650
-Connection ~ 4200 3650
-Wire Wire Line
-	4200 3650 4350 3650
 Text HLabel 4350 3850 2    50   Input ~ 0
 B02
-Wire Wire Line
-	4100 3850 4200 3850
-Wire Wire Line
-	4100 3950 4200 3950
-Wire Wire Line
-	4200 3950 4200 3850
-Connection ~ 4200 3850
-Wire Wire Line
-	4200 3850 4350 3850
 $Comp
 L power:GND #PWR0110
@@
 Wire Wire Line
 	5150 3950 5325 3950
+Wire Wire Line
+	4100 3150 4200 3150
+Wire Wire Line
+	4100 3250 4200 3250
+Wire Wire Line
+	4200 3250 4200 3150
+Connection ~ 4200 3150
+Wire Wire Line
+	4200 3150 4350 3150
+Wire Wire Line
+	4200 3350 4200 3450
+Wire Wire Line
+	4100 3350 4200 3350
+Wire Wire Line
+	4200 3350 4350 3350
+Connection ~ 4200 3350
+Wire Wire Line
+	4100 3650 4200 3650
+Wire Wire Line
+	4100 3750 4200 3750
+Wire Wire Line
+	4200 3750 4200 3650
+Connection ~ 4200 3650
+Wire Wire Line
+	4200 3650 4350 3650
+Wire Wire Line
+	4100 3850 4200 3850
+Wire Wire Line
+	4100 3950 4200 3950
+Wire Wire Line
+	4200 3950 4200 3850
+Connection ~ 4200 3850
+Wire Wire Line
+	4200 3850 4350 3850
 $EndSCHEMATC

Commit message: deel1routingpcb
Connections:
- net AIN1: now also MOTOR_DRIVER_IC1.22 (AIN2); no longer MOTOR_DRIVER_IC1.21 (AIN1)
- net AIN2: now also MOTOR_DRIVER_IC1.21 (AIN1); no longer MOTOR_DRIVER_IC1.22 (AIN2)
- net CIN1: now also MOTOR_DRIVER_IC2.22 (AIN2); no longer MOTOR_DRIVER_IC2.21 (AIN1)
- net CIN2: now also MOTOR_DRIVER_IC2.21 (AIN1); no longer MOTOR_DRIVER_IC2.22 (AIN2)
Changed lines of the file:
@@
 	2725 3450 2900 3450
 Text HLabel 2725 3750 0    50   Input ~ 0
+AIN1
+Text HLabel 2725 3650 0    50   Input ~ 0
 AIN2
-Text HLabel 2725 3650 0    50   Input ~ 0
-AIN1
 Wire Wire Line
 	2725 3650 2900 3650
@@
 	5150 3450 5325 3450
 Text HLabel 5150 3750 0    50   Input ~ 0
+CIN1
+Text HLabel 5150 3650 0    50   Input ~ 0
 CIN2
-Text HLabel 5150 3650 0    50   Input ~ 0
-CIN1
 Wire Wire Line
 	5150 3650 5325 3650
