File: pcbProject/Arduino_Uno_R3_From_Scratch.kicad_pcb (KiCad board)
At the start: 2 copper layers, 64.8 x 81.3 mm, 61 parts, among them J1 INTERRUPT, J2 STBY, P1 Power Header, P2 P2 Analog Header (AD), P3 Digital Header 02 (IOH) P3, P4 Digital Header 01 (IOL), P5 GND, P6 +5V, SW1 RESET_SWITCH, U1 NCP1117, U2 ATmega328P-AU, U3 LP2985-33DBVR, Y1 CSTCE16MOV53-R0

Commit message: pcbAfgewerktVersie1
volledig afgewerkte pcb 1e versie
Parts:
- IO_Expander (IC2): renamed from IO_Expander1
- MA-1A1: value MA-2B -> MA
- MB-1A1: value MB-2B -> MB
- MC-1A1: value MC-2B -> MC
- MD-1A1: value MD-2B -> MD
- renumbered LED6 to D3(PWM), LED5 to D5(PWM), LED4 to D6(PWM), LED3 to D9(PWM), GND1 to GND
Connections:
- P2 pad 7: /Headers/ARD_AN6 -> /ATMEGA328P/ARD_AN6
- P2 pad 8: /ATMEGA328P/ARD_AN6 -> /ATMEGA328P/ARD_AN7
- SW1 pad 3: (no net) -> GND
- SW1 pad 4: (no net) -> /ATMEGA328P/328P_RESET
- U2 pad 22: /Headers/ARD_AN6 -> /ATMEGA328P/ARD_AN7
Routing:
- net /ATMEGA328P/ARD_AN7: track 0.00 -> 45.1 mm
- net /Headers/ARD_AN6: track 42.5 -> 0.00 mm
- net /ATMEGA328P/328P_RESET: track 119.6 -> 133.3 mm, vias 0 -> 2
- net /ATMEGA328P/ARD_AN6: track 39.4 -> 38.4 mm
- net /ATMEGA328P/ARD_AN5/SCL: track 144.7 -> 145.5 mm
- net GND: track 588.2 -> 588.0 mm, vias 5 -> 6
- added copper zone on B.Cu, net /DecouplingCapacitors/VM
- added copper zone on B.Cu, net 5V_LDO
Other:
- board text added: "10"
- board text added: "11"
- board text added: "12"
- board text added: "3V3"
- board text added: "4"
- board text added: "5"
- board text added: "5V"
- board text added: "6"
- board text added: "7"
- board text added: "9"
- board text added: "A0"
- board text added: "A1"
- board text added: "A2"
- board text added: "A3"
- board text added: "A4"
- board text added: "A5"
- board text added: "A6"
- board text added: "A7"
- board text added: "AREF"
- board text added: "D0"
- board text added: "D1"
- board text added: "D2"
- board text added: "D4"
- board text added: "D7"
- board text added: "D8"
- board text added: "GND"
- board text added: "INT1"
- board text added: "INT2"
- board text added: "MISO"
- board text added: "MOSI"
- board text added: "RST"
- board text added: "SCK"
- board text added: "SCL"
- board text added: "SDA"
- board text added: "SPI_SS"
- board text added: "STBY"
