File: pcbProject/Arduino_Uno_R3_From_Scratch.kicad_pcb (KiCad board)
At the start: 2 copper layers, 61 parts, among them J1 INTERRUPT, J2 STBY, P1 Power Header, P2 P2 Analog Header (AD), P3 Digital Header 02 (IOH) P3, P4 Digital Header 01 (IOL), P5 GND, P6 +5V, SW1 RESET_SWITCH, U1 NCP1117, U2 ATmega328P-AU, U3 LP2985-33DBVR, Y1 CSTCE16MOV53-R0

Commit message: nogwatrouting
Parts:
- moved J2 172.9 mm to (118.5, 160.8), turned to 180 degrees
- moved R5 105.8 mm to (114.7, 157.0), turned to 90 degrees
- moved R6 94.8 mm to (103.4, 93.3), turned to 270 degrees
- moved P3 94.0 mm to (116.3, 122.6), turned to 180 degrees
- moved R7 87.3 mm to (105.9, 93.3), turned to 270 degrees
- moved P2 59.1 mm to (116.1, 98.3), turned to 180 degrees
- moved P4 45.6 mm to (82.9, 93.2)
- moved LED6 36.6 mm to (96.0, 115.6)
- moved R4 36.6 mm to (96.1, 120.3)
- moved LED3 35.4 mm to (104.4, 115.6)
- moved R1 35.4 mm to (104.2, 120.3)
- moved LED5 35.3 mm to (99.1, 115.6)
- moved R3 35.3 mm to (98.8, 120.3)
- moved LED1 35.1 mm to (92.6, 115.6)
- moved R10 35.1 mm to (92.6, 120.3)
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Routing:
- net /ATMEGA328P/ARD_DIG3: track 0.00 -> 39.4 mm
- net /ATMEGA328P/ARD_AN6: track 0.00 -> 38.3 mm
- net /Headers/ARD_AN6: track 0.00 -> 30.9 mm
- net /MotorDriver/B02: track 0.65 -> 24.3 mm
- net /ATMEGA328P/ARD_AN5/SCL: track 13.0 -> 36.2 mm
- net /MotorDriver/STBY: track 0.00 -> 22.4 mm
- net /ATMEGA328P/ARD_DIG10/SPI_SS: track 0.00 -> 19.9 mm
- net 5V_LDO: track 128.1 -> 147.8 mm
- net /ATMEGA328P/ARD_AN4/SDA: track 14.0 -> 33.1 mm
- net /ATMEGA328P/328P_RESET: track 0.00 -> 18.1 mm
- net 328P_ICSP_MOSI: track 0.00 -> 17.6 mm
- net /ATMEGA328P/ARD_AN3: track 0.00 -> 15.9 mm
- net 328P_ICSP_MISO: track 0.00 -> 15.9 mm
- net 328P_ICSP_SCK: track 0.00 -> 14.2 mm
- net /ATMEGA328P/ARD_AN2: track 0.00 -> 13.9 mm
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
Commit message: pcb
Parts:
- moved P6 170.5 mm to (87.8, 66.2)
- moved P5 157.2 mm to (81.4, 72.5)
- moved C17 90.0 mm to (97.4, 140.7), turned to 180 degrees
- moved C4 82.3 mm to (124.3, 122.2), turned to 270 degrees
- moved C12 70.8 mm to (104.8, 117.9), turned to 180 degrees
- moved C15 65.6 mm to (93.5, 116.2), turned to 180 degrees
- moved C18 65.6 mm to (93.5, 119.5), turned to 180 degrees
- moved C6 64.5 mm to (102.9, 99.7), turned to 270 degrees
- moved C16 64.4 mm to (104.8, 121.3), turned to 180 degrees
- moved C13 54.2 mm to (115.4, 111.8), turned to 90 degrees
- moved R11 51.9 mm to (85.6, 113.5)
- moved C5 51.5 mm to (88.6, 117.7)
- moved C7 49.5 mm to (81.9, 112.4)
- moved U3 49.5 mm to (98.6, 99.6)
- moved C11 46.9 mm to (100.6, 104.9)
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Connections:
- P1 pad 1: /ATMEGA328P/328P_RESET -> GND
- P1 pad 2: 3V3_LDO -> GND
- P1 pad 3: 5V_LDO -> 3V3_LDO
- P1 pad 4: GND -> 3V3_LDO
- P1 pad 5: GND -> 5V_LDO
- P1 pad 6: 3V3_LDO -> /ATMEGA328P/328P_RESET
Routing:
- net GND: track 177.6 -> 295.1 mm
- net 5V_LDO: track 147.8 -> 211.0 mm
- net /ATMEGA328P/ARD_DIG7: track 0.00 -> 48.0 mm
- net /ATMEGA328P/ARD_DIG8: track 0.00 -> 47.4 mm
- net /MotorDriver/STBY: track 22.4 -> 62.0 mm
- net /DecouplingCapacitors/VM: track 44.7 -> 73.1 mm
- net /ATMEGA328P/ARD_DIG0: track 0.00 -> 23.2 mm
- net /ATMEGA328P/ARD_DIG1: track 0.00 -> 21.2 mm
- net 328P_ICSP_MOSI: track 17.6 -> 38.7 mm
- net /ATMEGA328P/ARD_DIG2: track 0.00 -> 20.1 mm
- net 328P_ICSP_SCK: track 14.2 -> 32.8 mm
- net 328P_ICSP_MISO: track 15.9 -> 29.2 mm
- net /ATMEGA328P/328P_RESET: track 18.1 -> 30.6 mm
- net 3V3_LDO: track 35.5 -> 28.4 mm
- net /ATMEGA328P/ARD_DIG3: track 39.4 -> 36.1 mm
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
Commit message: pcb wijziging
Parts:
- moved P2 7.50 mm to (133.9, 85.1)
- moved C14 7.23 mm to (128.9, 90.0)
- moved P6 7.00 mm to (88.3, 73.2)
- moved U2 6.99 mm to (120.3, 90.4)
- moved R17 6.99 mm to (112.6, 94.2)
- moved R1 6.60 mm to (123.3, 106.2)
- moved R2 6.60 mm to (119.1, 106.2)
- moved R3 6.60 mm to (114.4, 106.2)
- moved R4 6.60 mm to (110.1, 106.2)
- moved LED3 6.60 mm to (123.6, 101.5)
- moved LED4 6.60 mm to (119.3, 101.5)
- moved LED5 6.60 mm to (114.7, 101.5)
- moved LED6 6.60 mm to (110.0, 101.5)
- moved C2 6.04 mm to (95.8, 92.8)
- moved Y1 3.43 mm to (107.8, 88.1)
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Routing:
- net GND: track 295.1 -> 328.0 mm
- net /Headers/ARD_AN6: track 30.9 -> 0.00 mm
- net /ATMEGA328P/ARD_AN6: track 38.3 -> 11.0 mm
- net /ATMEGA328P/ARD_AN5/SCL: track 36.2 -> 13.9 mm
- net /ATMEGA328P/ARD_DIG1: track 21.2 -> 6.16 mm
- net /ATMEGA328P/ARD_DIG2: track 20.1 -> 5.19 mm
- net /ATMEGA328P/328P_RESET: track 30.6 -> 44.5 mm
- net /ATMEGA328P/ARD_AN4/SDA: track 33.1 -> 19.9 mm
- net /ATMEGA328P/ARD_AN3: track 15.9 -> 3.04 mm
- net /ATMEGA328P/ARD_AN2: track 13.9 -> 1.22 mm
- net /ATMEGA328P/ARD_AN1: track 11.3 -> 0.00 mm
- net /ATMEGA328P/ARD_AN0: track 10.5 -> 0.00 mm
- net /ATMEGA328P/ARD_DIG3: track 36.1 -> 26.6 mm
- net Net-(R17-Pad2): track 12.6 -> 3.54 mm
- net /ATMEGA328P/ARD_DIG7: track 48.0 -> 56.5 mm
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
Commit message: bijna klaar pcb
nog enkele andere planes toevoegen
Parts:
- SW1: footprint Button_Switch_SMD:SW_SPST_PTS645 -> eigenfootprint:SW_SPST_PTS645_aangepast
- moved SW1 17.8 mm to (130.4, 81.4), turned to 180 degrees
- moved P2 13.6 mm to (126.2, 73.8), turned to 270 degrees
- moved R16 13.0 mm to (116.8, 79.0)
- moved R6 6.95 mm to (120.8, 81.9), turned to 0 degrees
- moved R7 5.68 mm to (120.8, 79.4), turned to 0 degrees
- moved P5 2.36 mm to (85.7, 71.8)
- moved P3 2.17 mm to (133.6, 104.0)
- moved P6 2.07 mm to (89.8, 71.8)
- moved ICSP2 1.80 mm to (133.0, 109.2)
- moved C14 1.40 mm to (128.8, 91.4), turned to 90 degrees
Connections:
- SW1 pad 1: /ATMEGA328P/328P_RESET -> GND
Routing:
- net GND: track 328.0 -> 588.2 mm, vias 0 -> 5
- net 5V_LDO: track 204.7 -> 382.5 mm, vias 0 -> 5
- net /ATMEGA328P/ARD_AN5/SCL: track 13.9 -> 144.7 mm, vias 0 -> 2
- net /ATMEGA328P/ARD_DIG6: track 6.27 -> 106.6 mm, vias 0 -> 2
- net /DecouplingCapacitors/VM: track 73.1 -> 157.3 mm, vias 0 -> 4
- net /ATMEGA328P/328P_RESET: track 44.5 -> 119.6 mm
- net /ATMEGA328P/ARD_AN4/SDA: track 19.9 -> 89.3 mm, vias 0 -> 2
- net /ATMEGA328P/ARD_DIG5: track 10.1 -> 61.7 mm, vias 0 -> 2
- net /ATMEGA328P/ARD_DIG3: track 26.6 -> 76.9 mm, vias 0 -> 4
- net /Headers/ARD_AN6: track 0.00 -> 42.5 mm
- net /ATMEGA328P/ARD_DIG9: track 9.62 -> 49.4 mm, vias 0 -> 2
- net /ATMEGA328P/ARD_AN6: track 11.0 -> 39.4 mm, vias 0 -> 1
- net /ATMEGA328P/ARD_AN3: track 3.04 -> 26.6 mm
- net /ATMEGA328P/ARD_AN1: track 0.00 -> 22.4 mm
- net /ATMEGA328P/ARD_DIG4: track 0.00 -> 22.2 mm
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- added copper zone on B.Cu, net GND
- added copper zone on F.Cu, net GND
Other:
- board outline added: 64.8 x 81.3 mm
