File: pcbProject/ATMEGA328P.sch (KiCad schematic (older format))
At the start: 8 parts, among them SW1 RESET_SWITCH, U5 ATMEGA328P, X2 CSTCE16MOV53-R0

Commit message: pcbarduino
THT atmega aangepast naar smd en volledig schema afgewerkt
Parts:
- removed U5: ATMEGA328P, ~, symbol MFN_Atmel:ATMEGA328P-PU
- added U?: ATmega328P-AU, Package_QFP:TQFP-32_7x7mm_P0.8mm, symbol MCU_Microchip_ATmega:ATmega328P-AU
Connections:
- wire segments 80 -> 88
Other:
- moved on the sheet: C14, C15, ICSP2, R16, R17, SW1, X2

Commit message: af
Parts:
- gave numbers to parts that had none: 1
Changed lines of the file:
@@
 	4925 2350 4925 2450
 $Comp
-L power:GND #PWR?
+L power:GND #PWR08
 U 1 1 5C7DB759
 P 10475 3800
-F 0 "#PWR?" H 10475 3550 50  0001 C CNN
+F 0 "#PWR08" H 10475 3550 50  0001 C CNN
 F 1 "GND" H 10480 3627 50  0000 C CNN
 F 2 "" H 10475 3800 50  0001 C CNN
@@
 	10475 3800 10475 3475
 $Comp
-L MCU_Microchip_ATmega:ATmega328P-AU U?
+L MCU_Microchip_ATmega:ATmega328P-AU U2
 U 1 1 5C76D532
 P 4825 3950
-F 0 "U?" H 4825 2364 50  0000 C CNN
+F 0 "U2" H 4825 2364 50  0000 C CNN
 F 1 "ATmega328P-AU" H 4825 2273 50  0000 C CNN
 F 2 "Package_QFP:TQFP-32_7x7mm_P0.8mm" H 4825 3950 50  0001 C CIN
@@
 	2850 2750 4225 2750
 $Comp
-L power:GND #PWR?
+L power:GND #PWR03
 U 1 1 5C83660C
 P 4825 5900
-F 0 "#PWR?" H 4825 5650 50  0001 C CNN
+F 0 "#PWR03" H 4825 5650 50  0001 C CNN
 F 1 "GND" H 4830 5727 50  0000 C CNN
 F 2 "" H 4825 5900 50  0001 C CNN

Commit message: schema Afgewerkt
Connections:
- net ARD_AN6: now reaches U2.19 (ADC6)
- net ARD_AN7: now reaches U2.22 (ADC7)
Changed lines of the file:
@@
 Wire Wire Line
 	1975 3550 1975 3275
+Text HLabel 4000 2950 0    40   Input ~ 0
+ARD_AN6
+Text HLabel 4000 3050 0    40   Input ~ 0
+ARD_AN7
+Wire Wire Line
+	4000 2950 4225 2950
+Wire Wire Line
+	4000 3050 4225 3050
 $EndSCHEMATC

Commit message: deel1routingpcb
Parts:
- removed X2: CSTCE16MOV53-R0, ~, symbol Arduino_Uno_R3_From_Scratch:CERAMIC_RESONATOR
- added Y1: CSTCE16MOV53-R0, Crystal:Crystal_SMD_HC49-SD, symbol Device:Crystal
- C14, C15: footprint ~ -> Capacitor_SMD:C_1206_3216Metric
- ICSP2: footprint ~ -> Connector_PinSocket_2.54mm:PinSocket_2x03_P2.54mm_Vertical
- R16, R17: footprint ~ -> Resistor_SMD:R_1206_3216Metric
- SW1: footprint (none) -> Button_Switch_SMD:SW_SPST_PTS645
Connections:
- net at R17.1, U2.8 (XTAL2/PB7): now also Y1.2
- net at R17.2, U2.7 (XTAL1/PB6): now also Y1.1
Changed lines of the file:
@@
 F 0 "ICSP2" H 1900 1550 50  0000 C CNN
 F 1 "M20-9980346" H 1900 1100 40  0000 C CNN
-F 2 "~" H 1900 1300 60  0000 C CNN
+F 2 "Connector_PinSocket_2.54mm:PinSocket_2x03_P2.54mm_Vertical" H 1900 1300 60  0000 C CNN
 F 3 "http://cdn.harwin.com/pdfs/M20-998.pdf" H 1900 1300 60  0001 C CNN
 F 4 "6 CONTACT(S), MALE, STRAIGHT TWO PART BOARD CONNECTOR" H 1900 1300 60  0001 C CNN "Characteristics"
@@
 F 0 "SW1" V 1350 2725 60  0000 C CNN
 F 1 "RESET_SWITCH" V 1650 2975 60  0000 C CNN
-F 2 "" H 1500 2425 60  0001 C CNN
+F 2 "Button_Switch_SMD:SW_SPST_PTS645" H 1500 2425 60  0001 C CNN
 F 3 "http://industrial.panasonic.com/www-data/pdf/ATK0000/ATK0000CE28.pdf" H 1500 2425 60  0001 C CNN
 F 4 "SWITCH TACTILE SPST-NO 0.02A 15V" H 1500 2425 60  0001 C CNN "Characteristics"
@@
 	1    0    0    -1
 $EndComp
-$Comp
-L Arduino_Uno_R3_From_Scratch:CERAMIC_RESONATOR X2
-U 1 1 5614A1DB
-P 10000 3475
-F 0 "X2" V 10075 3375 50  0000 R CNN
-F 1 "CSTCE16MOV53-R0" V 9925 3375 40  0000 R CNN
-F 2 "~" H 10000 3475 60  0000 C CNN
-F 3 "http://www.murata.com/~/media/webrenewal/support/library/catalog/products/timingdevice/ceralock/p16e.ashx" H 10000 3475 60  0001 C CNN
-F 4 "CER RESONATOR 16.0MHZ SMD" H 10000 3475 60  0001 C CNN "Characteristics"
-F 5 "ATMEGA328P Oscillator" H 10000 3475 60  0001 C CNN "Description"
-F 6 "Murata" H 10000 3475 60  0001 C CNN "MFN"
-F 7 "CSTCE16M0V53-R0" H 10000 3475 60  0001 C CNN "MFP"
-F 8 "SMD" H 10000 3475 60  0001 C CNN "Package ID"
-F 9 "ANY" H 10000 3475 60  0001 C CNN "Source"
-F 10 "Y" H 10000 3475 60  0001 C CNN "Critical"
-F 11 "328P_Sub" H 10000 3475 60  0001 C CNN "Subsystem"
-F 12 "~" H 10000 3475 60  0001 C CNN "Notes"
-	1    10000 3475
-	0    -1   -1   0
-$EndComp
 Wire Wire Line
 	9950 3975 9600 3975
 Wire Wire Line
-	9950 3975 9950 3875
-Wire Wire Line
-	9950 3075 9950 2975
-Wire Wire Line
 	9950 2975 9600 2975
-Wire Wire Line
-	10200 3475 10475 3475
 Text Notes 7025 1050 0    40   ~ 0
 Atmel Appnote: AVR042 - AVR Hardware Design Considerations\nhttp://www.atmel.com/Images/Atmel-2521-AVR-Hardware-Design-Considerations_ApplicationNote_AVR042.pdf\n\nRefer to this for PCB layout information
@@
 F 0 "C14" H 2900 3250 40  0000 L CNN
 F 1 "0.1 uF" H 2900 3050 40  0000 L CNN
-F 2 "~" H 2888 3000 30  0000 C CNN
+F 2 "Capacitor_SMD:C_1206_3216Metric" H 2888 3000 30  0000 C CNN
 F 3 "http://images.ihscontent.net/vipimages/VipMasterIC/IC/KEME/KEMES10043/KEMES10043-1.pdf" H 2850 3150 60  0001 C CNN
 F 4 "CAPACITOR, CERAMIC, MULTILAYER, 100 V, X7R, 0.1 uF, SURFACE MOUNT, 0805, CHIP, ROHS COMPLIANT" H 2850 3150 60  0001 C CNN "Characteristics"
@@
 F 0 "C15" H 2025 3225 40  0000 L CNN
 F 1 "0.1 uF" H 2025 3025 40  0000 L CNN
-F 2 "~" H 2013 2975 30  0000 C CNN
+F 2 "Capacitor_SMD:C_1206_3216Metric" H 2013 2975 30  0000 C CNN
 F 3 "http://images.ihscontent.net/vipimages/VipMasterIC/IC/KEME/KEMES10043/KEMES10043-1.pdf" H 1975 3125 60  0001 C CNN
 F 4 "CAPACITOR, CERAMIC, MULTILAYER, 100 V, X7R, 0.1 uF, SURFACE MOUNT, 0805, CHIP, ROHS COMPLIANT" H 1975 3125 60  0001 C CNN "Characteristics"
@@
 F 0 "R16" V 3080 1650 40  0000 C CNN
 F 1 "10K" V 3007 1651 40  0000 C CNN
-F 2 "~" V 2930 1650 30  0000 C CNN
+F 2 "Resistor_SMD:R_1206_3216Metric" V 2930 1650 30  0000 C CNN
 F 3 "http://images.ihscontent.net/vipimages/VipMasterIC/IC/VISH/VISHS75859/VISHS75859-1.pdf" H 3000 1650 30  0001 C CNN
 F 4 "RESISTOR, METAL GLAZE/THICK FILM, 0.125W, 5%, 200ppm, 10000ohm, SURFACE MOUNT, 0805" H 3000 1650 60  0001 C CNN "Characteristics"
@@
 F 0 "R17" H 9675 3425 40  0000 L CNN
 F 1 "1M" V 9600 3475 40  0000 C CNN
-F 2 "~" V 9530 3475 30  0000 C CNN
+F 2 "Resistor_SMD:R_1206_3216Metric" V 9530 3475 30  0000 C CNN
 F 3 "http://www.vishay.com/docs/20035/dcrcwe3.pdf" H 9600 3475 30  0001 C CNN
 F 4 "RES SMD 1M OHM 1% 1/8W 0805" H 9600 3475 60  0001 C CNN "Characteristics"
@@
 	4925 2350 4925 2450
 $Comp
-L power:GND #PWR08
-U 1 1 5C7DB759
-P 10475 3800
-F 0 "#PWR08" H 10475 3550 50  0001 C CNN
-F 1 "GND" H 10480 3627 50  0000 C CNN
-F 2 "" H 10475 3800 50  0001 C CNN
-F 3 "" H 10475 3800 50  0001 C CNN
-	1    10475 3800
-	1    0    0    -1
-$EndComp
-Wire Wire Line
-	10475 3800 10475 3475
-$Comp
 L MCU_Microchip_ATmega:ATmega328P-AU U2
 U 1 1 5C76D532
@@
 Wire Wire Line
 	4000 3050 4225 3050
+$Comp
+L Device:Crystal Y1
+U 1 1 5C9F065B
+P 9950 3475
+F 0 "Y1" V 9904 3606 50  0000 L CNN
+F 1 "CSTCE16MOV53-R0" V 9995 3606 50  0000 L CNN
+F 2 "Crystal:Crystal_SMD_HC49-SD" H 9950 3475 50  0001 C CNN
+F 3 "~" H 9950 3475 50  0001 C CNN
+	1    9950 3475
+	0    1    1    0
+$EndComp
+Wire Wire Line
+	9950 3625 9950 3975
+Wire Wire Line
+	9950 2975 9950 3325
 $EndSCHEMATC

Commit message: bijna klaar pcb
nog enkele andere planes toevoegen
Parts:
- SW1: footprint Button_Switch_SMD:SW_SPST_PTS645 -> eigenfootprint:SW_SPST_PTS645_aangepast
Changed lines of the file:
@@
 F 0 "SW1" V 1350 2725 60  0000 C CNN
 F 1 "RESET_SWITCH" V 1650 2975 60  0000 C CNN
-F 2 "Button_Switch_SMD:SW_SPST_PTS645" H 1500 2425 60  0001 C CNN
+F 2 "eigenfootprint:SW_SPST_PTS645_aangepast" H 1500 2425 60  0001 C CNN
 F 3 "http://industrial.panasonic.com/www-data/pdf/ATK0000/ATK0000CE28.pdf" H 1500 2425 60  0001 C CNN
 F 4 "SWITCH TACTILE SPST-NO 0.02A 15V" H 1500 2425 60  0001 C CNN "Characteristics"

Commit message: NIEUWE PCB VERSIE
Parts:
- added C19, C20: 22p, Capacitor_SMD:C_0805_2012Metric, symbol Device:C
Connections:
- net GND: now also C19.2, C20.2
- net at R17.1, U2.8 (XTAL2/PB7), Y1.2: now also C20.1
- net at R17.2, U2.7 (XTAL1/PB6), Y1.1: now also C19.1
Changed lines of the file:
@@
 $EndComp
 Wire Wire Line
-	9950 3625 9950 3975
+	9950 3625 9950 3700
 Wire Wire Line
 	9950 2975 9950 3325
+$Comp
+L Device:C C20
+U 1 1 5C89A715
+P 10350 3850
+F 0 "C20" H 10465 3896 50  0000 L CNN
+F 1 "22p" H 10465 3805 50  0000 L CNN
+F 2 "Capacitor_SMD:C_0805_2012Metric" H 10388 3700 50  0001 C CNN
+F 3 "~" H 10350 3850 50  0001 C CNN
+	1    10350 3850
+	1    0    0    -1
+$EndComp
+$Comp
+L Device:C C19
+U 1 1 5C89A779
+P 10350 3125
+F 0 "C19" H 10465 3171 50  0000 L CNN
+F 1 "22p" H 10465 3080 50  0000 L CNN
+F 2 "Capacitor_SMD:C_0805_2012Metric" H 10388 2975 50  0001 C CNN
+F 3 "~" H 10350 3125 50  0001 C CNN
+	1    10350 3125
+	1    0    0    -1
+$EndComp
+Wire Wire Line
+	9950 2975 10350 2975
+Connection ~ 9950 2975
+Wire Wire Line
+	9950 3700 10350 3700
+Connection ~ 9950 3700
+Wire Wire Line
+	9950 3700 9950 3975
+$Comp
+L power:GND #PWR09
+U 1 1 5C89ED8F
+P 10350 4050
+F 0 "#PWR09" H 10350 3800 50  0001 C CNN
+F 1 "GND" H 10355 3877 50  0000 C CNN
+F 2 "" H 10350 4050 50  0001 C CNN
+F 3 "" H 10350 4050 50  0001 C CNN
+	1    10350 4050
+	1    0    0    -1
+$EndComp
+$Comp
+L power:GND #PWR08
+U 1 1 5C89EDC5
+P 10350 3325
+F 0 "#PWR08" H 10350 3075 50  0001 C CNN
+F 1 "GND" H 10355 3152 50  0000 C CNN
+F 2 "" H 10350 3325 50  0001 C CNN
+F 3 "" H 10350 3325 50  0001 C CNN
+	1    10350 3325
+	1    0    0    -1
+$EndComp
+Wire Wire Line
+	10350 3325 10350 3275
+Wire Wire Line
+	10350 4050 10350 4000
 $EndSCHEMATC
