File: pcbProject/PullUpResisters.sch (KiCad schematic (older format))
At the start: 5 parts

Commit message: deel1routingpcb
Parts:
- R5, R6, R7, R8, R9: footprint (none) -> Resistor_SMD:R_1206_3216Metric
Changed lines of the file:
@@
 F 0 "R9" V 4675 3300 50  0000 C CNN
 F 1 "10k" V 4509 3125 50  0000 C CNN
-F 2 "" V 4555 3125 50  0001 C CNN
+F 2 "Resistor_SMD:R_1206_3216Metric" V 4555 3125 50  0001 C CNN
 F 3 "~" H 4625 3125 50  0001 C CNN
 	1    4625 3125
@@
 F 0 "R8" V 4675 3600 50  0000 C CNN
 F 1 "10k" V 4509 3425 50  0000 C CNN
-F 2 "" V 4555 3425 50  0001 C CNN
+F 2 "Resistor_SMD:R_1206_3216Metric" V 4555 3425 50  0001 C CNN
 F 3 "~" H 4625 3425 50  0001 C CNN
 	1    4625 3425
@@
 F 0 "R7" V 4675 3925 50  0000 C CNN
 F 1 "10k" V 4509 3750 50  0000 C CNN
-F 2 "" V 4555 3750 50  0001 C CNN
+F 2 "Resistor_SMD:R_1206_3216Metric" V 4555 3750 50  0001 C CNN
 F 3 "~" H 4625 3750 50  0001 C CNN
 	1    4625 3750
@@
 F 0 "R6" V 4675 4225 50  0000 C CNN
 F 1 "10k" V 4509 4050 50  0000 C CNN
-F 2 "" V 4555 4050 50  0001 C CNN
+F 2 "Resistor_SMD:R_1206_3216Metric" V 4555 4050 50  0001 C CNN
 F 3 "~" H 4625 4050 50  0001 C CNN
 	1    4625 4050
@@
 F 0 "R5" V 4675 4550 50  0000 C CNN
 F 1 "10k" V 4509 4375 50  0000 C CNN
-F 2 "" V 4555 4375 50  0001 C CNN
+F 2 "Resistor_SMD:R_1206_3216Metric" V 4555 4375 50  0001 C CNN
 F 3 "~" H 4625 4375 50  0001 C CNN
 	1    4625 4375

Commit message: PCB versie3
Aanpassingen tips coach --> veel gewijzigd
Parts:
- R5, R6, R7, R8, R9: footprint Resistor_SMD:R_1206_3216Metric -> Resistor_SMD:R_1206_3216Metric_Pad1.42x1.75mm_HandSolder
Changed lines of the file:
@@
 F 0 "R9" V 4675 3300 50  0000 C CNN
 F 1 "10k" V 4509 3125 50  0000 C CNN
-F 2 "Resistor_SMD:R_1206_3216Metric" V 4555 3125 50  0001 C CNN
+F 2 "Resistor_SMD:R_1206_3216Metric_Pad1.42x1.75mm_HandSolder" V 4555 3125 50  0001 C CNN
 F 3 "~" H 4625 3125 50  0001 C CNN
 	1    4625 3125
@@
 F 0 "R8" V 4675 3600 50  0000 C CNN
 F 1 "10k" V 4509 3425 50  0000 C CNN
-F 2 "Resistor_SMD:R_1206_3216Metric" V 4555 3425 50  0001 C CNN
+F 2 "Resistor_SMD:R_1206_3216Metric_Pad1.42x1.75mm_HandSolder" V 4555 3425 50  0001 C CNN
 F 3 "~" H 4625 3425 50  0001 C CNN
 	1    4625 3425
@@
 F 0 "R7" V 4675 3925 50  0000 C CNN
 F 1 "10k" V 4509 3750 50  0000 C CNN
-F 2 "Resistor_SMD:R_1206_3216Metric" V 4555 3750 50  0001 C CNN
+F 2 "Resistor_SMD:R_1206_3216Metric_Pad1.42x1.75mm_HandSolder" V 4555 3750 50  0001 C CNN
 F 3 "~" H 4625 3750 50  0001 C CNN
 	1    4625 3750
@@
 F 0 "R6" V 4675 4225 50  0000 C CNN
 F 1 "10k" V 4509 4050 50  0000 C CNN
-F 2 "Resistor_SMD:R_1206_3216Metric" V 4555 4050 50  0001 C CNN
+F 2 "Resistor_SMD:R_1206_3216Metric_Pad1.42x1.75mm_HandSolder" V 4555 4050 50  0001 C CNN
 F 3 "~" H 4625 4050 50  0001 C CNN
 	1    4625 4050
@@
 F 0 "R5" V 4675 4550 50  0000 C CNN
 F 1 "10k" V 4509 4375 50  0000 C CNN
-F 2 "Resistor_SMD:R_1206_3216Metric" V 4555 4375 50  0001 C CNN
+F 2 "Resistor_SMD:R_1206_3216Metric_Pad1.42x1.75mm_HandSolder" V 4555 4375 50  0001 C CNN
 F 3 "~" H 4625 4375 50  0001 C CNN
 	1    4625 4375
